Commit message: Change max effort of motors

File: jsk_hand/dynamixel_detachable_hand/urdf/lhand.urdf (robot description, URDF)
Before this commit: robot lhand_robot, 2 links, 1 joints
Joints:
- joint lhand_joint: limit effort=0.92 velocity=6.8 -> effort=2.00 velocity=6.8

File: jsk_hand/dynamixel_detachable_hand/urdf/rhand.urdf (robot description, URDF)
Before this commit: robot rhand_robot, 2 links, 1 joints
Joints:
- joint rhand_joint: limit effort=0.92 velocity=6.8 -> effort=2.0 velocity=6.8

Commit message: 能動脱着対応

File: jsk_hand/dynamixel_detachable_hand/urdf/lhand.urdf (robot description, URDF)
Before this commit: robot lhand_robot, 2 links, 1 joints
Links:
- added link lhand_detach_link_0; visual box size=0.08 0.08 0.1
Joints:
- added joint lhand_detach_joint_0: type continuous, parent base_link, child lhand_detach_link_0, origin xyz=0.1 0 0.1 rpy=0 0 0, axis 0 1 0, limit effort=2.0 velocity=6.8

File: jsk_hand/dynamixel_detachable_hand/urdf/rhand.urdf (robot description, URDF)
Before this commit: robot rhand_robot, 2 links, 1 joints
Links:
- added link rhand_detach_link_0; visual box size=0.08 0.08 0.1
Joints:
- added joint rhand_detach_joint_0: type continuous, parent base_link, child rhand_detach_link_0, origin xyz=0.1 0 0.1 rpy=0 0 0, axis 0 1 0, limit effort=2.0 velocity=6.8
