Commit message: Add SURGENOID needle holder detachable model

File: jsk_hand/dynamixel_detachable_hand/urdf/lhand_detacher.urdf (robot description, URDF)
Before this commit: robot lhand_detacher_robot, 2 links, 1 joints
Links:
- removed link base_link
- added link lhand_base_link; visual box size=0.2 0.2 0.2
Joints:
- joint lhand_detach_joint_0: parent base_link -> lhand_base_link

File: jsk_hand/dynamixel_detachable_hand/urdf/lhand_gripper.urdf (robot description, URDF)
Before this commit: robot lhand_gripper_robot, 3 links, 2 joints
Links:
- removed link lhand_link
- added link lhand_bottom_spacer3300a_1, mass 0.00617072; collision mesh filename=package://dynamixel_detachable_hand/meshes/nejineji_finger_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; visual mesh filename=package://dynamixel_detachable_hand/meshes/nejineji_finger_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
- added link lhand_finger_11, mass 0.0442481; collision mesh filename=package://dynamixel_detachable_hand/meshes/nejineji_finger_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; visual mesh filename=package://dynamixel_detachable_hand/meshes/nejineji_finger_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
- added link lhand_finger_13, mass 0.0442481; collision mesh filename=package://dynamixel_detachable_hand/meshes/nejineji_finger_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; visual mesh filename=package://dynamixel_detachable_hand/meshes/nejineji_finger_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
- added link lhand_pinion_1, mass 0.00261444; collision mesh filename=package://dynamixel_detachable_hand/meshes/nejineji_finger_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; visual mesh filename=package://dynamixel_detachable_hand/meshes/nejineji_finger_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
- added link lhand_screwlock_male_1, mass 0.0103795; collision mesh filename=package://dynamixel_detachable_hand/meshes/nejineji_finger_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; visual mesh filename=package://dynamixel_detachable_hand/meshes/nejineji_finger_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
- added link lhand_small_diameter_hornb_1, mass 0.000682303; collision mesh filename=package://dynamixel_detachable_hand/meshes/nejineji_finger_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; visual mesh filename=package://dynamixel_detachable_hand/meshes/nejineji_finger_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
- added link lhand_tip_link
- added link lhand_xl_xc_330_1_2, mass 0.0168537; collision mesh filename=package://dynamixel_detachable_hand/meshes/nejineji_finger_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; visual mesh filename=package://dynamixel_detachable_hand/meshes/nejineji_finger_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
- link lhand_base_link: mass None -> 0.0498606; geometry collision mesh filename=package://dynamixel_detachable_hand/meshes/nejineji_finger_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; visual mesh filename=package://dynamixel_detachable_hand/meshes/nejineji_finger_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
Joints:
- added joint lhand_buttom_spacer3300a_1__screwlock_male_1: type fixed, parent lhand_bottom_spacer3300a_1, child lhand_screwlock_male_1, origin xyz=-5.6e-06 0.007707033 -0.003298772 rpy=0 -1.570796301 0, axis -0 1 -0
- added joint lhand_finger_mimic_joint: type prismatic, parent lhand_base_link, child lhand_finger_13, origin xyz=0 0 0 rpy=0 -0 0, axis -1 0 0, limit lower=-0.05 upper=0 effort=10 velocity=3.14, mimic joint=lhand_joint multiplier=-1 offset=0
- added joint lhand_servo_and_case_simple_1__pinion_1: type fixed, parent lhand_base_link, child lhand_pinion_1, origin xyz=-6.95e-06 -7.0943e-05 0.005234895 rpy=-3.141592607 0 -0.09765488, axis -0 0 -1
- added joint lhand_servo_and_case_simple_1__small_diameter_hornb_1: type fixed, parent lhand_base_link, child lhand_small_diameter_hornb_1, origin xyz=-5.065e-06 0 0.000967784 rpy=0 0 -3.141592607, axis 0 1 0
- added joint lhand_servo_and_case_simple_1__xl_xc_330_1_2: type fixed, parent lhand_base_link, child lhand_xl_xc_330_1_2, origin xyz=-0.0067468 7.9755e-05 -0.015702072 rpy=0 0 -1.5707963, axis 0 0 -1
- added joint lhand_to_tip: type fixed, parent lhand_base_link, child lhand_tip_link, origin xyz=0 0 0.06743 rpy=0 0 0
- added joint lhand_xl_xc_330_1_2__buttom_spacer3300a_1: type fixed, parent lhand_xl_xc_330_1_2, child lhand_bottom_spacer3300a_1, origin xyz=7.9799e-05 0.003444766 -0.015364374 rpy=-1.5707963 0 3.141592607, axis 0 -1 0
- joint lhand_joint: axis 0 1 0 -> -1 0 0; child lhand_link -> lhand_finger_11; limit effort=2.00 velocity=6.8 -> lower=0 upper=0.05 effort=2.0 velocity=0.1; origin xyz=0 0 0.1 rpy=0 0 0 -> xyz=0 0 0 rpy=0 -0 0; type continuous -> prismatic

File: jsk_hand/dynamixel_detachable_hand/urdf/lhand_needle_holder.urdf (robot description, URDF)
Before this commit: robot lhand_needle_holder_robot, 9 links, 8 joints
Links:
- removed link lhand_SURGERY_CLAMP_01_1
- removed link lhand_SURGERY_CLAMP_ASSY_1
- removed link lhand_XL_XC_330_1
- removed link lhand_command_link
- removed link lhand_small_needle_hoder_base_1
- added link lhand_small_needle_holder_base_1, mass 0.020773; collision mesh filename=package://surgenoid_needle_holder_description/meshes/small_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; visual mesh filename=package://surgenoid_needle_holder_description/meshes/small_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
- added link lhand_surgery_clamp_01_1, mass 0.00562524; collision mesh filename=package://surgenoid_needle_holder_description/meshes/SURGER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; visual mesh filename=package://surgenoid_needle_holder_description/meshes/SURGER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
- added link lhand_surgery_clamp_assy_1, mass 0.00675555; collision mesh filename=package://surgenoid_needle_holder_description/meshes/SURGER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; visual mesh filename=package://surgenoid_needle_holder_description/meshes/SURGER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
- added link lhand_xl_xc_330_1, mass 0.0168532; collision mesh filename=package://surgenoid_needle_holder_description/meshes/XL_XC_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; visual mesh filename=package://surgenoid_needle_holder_description/meshes/XL_XC_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
- link lhand_detach_link_0: mass None -> 0.01
Joints:
- removed joint SURGERY_CLAMP_ASSY_1__SURGERY_CLAMP_01_1
- removed joint XL_XC_330_1__small_needle_holder_link1_1
- removed joint screwlock_male_hard_v2_1__small_needle_hoder_base_1
- removed joint small_needle_hoder_base_1__SURGERY_CLAMP_ASSY_1
- removed joint small_needle_hoder_base_1__XL_XC_330_1
- removed joint small_needle_holder_link1_1__small_needle_holder_link2_1
- added joint lhand_holder_base_to_clamp: type fixed, parent lhand_small_needle_holder_base_1, child lhand_surgery_clamp_assy_1, origin xyz=-0.037277901 0.011289345 -0.004030915 rpy=0 0 -3.0922928, axis 0 0 -1
- added joint lhand_holder_base_to_motor: type fixed, parent lhand_small_needle_holder_base_1, child lhand_xl_xc_330_1, origin xyz=0.038688034 -0.006248738 0.011774486 rpy=-3.141592607 0 1.5707963, axis 0 0 -1
- added joint lhand_holder_jaw_joint: type revolute, parent lhand_surgery_clamp_assy_1, child lhand_surgery_clamp_01_1, origin xyz=0.040124645 -0.00714826 0.001320943 rpy=0 0 3.0922928, axis 0 0 -1, limit lower=-0.29662 upper=0.44772 effort=10 velocity=3.14, mimic joint=lhand_joint multiplier=0.581031 offset=0
- added joint lhand_holder_screw_to_base: type fixed, parent lhand_base_link, child lhand_small_needle_holder_base_1, origin xyz=-0.009065668 -0.000168333 -0.015571405 rpy=-6.327e-06 -2.654e-06 3.141589, axis 0 0 1
- added joint lhand_holder_tip_joint: type revolute, parent lhand_small_needle_holder_link1_1, child lhand_small_needle_holder_link2_1, origin xyz=0.020772397 0.033007689 -0.017 rpy=0 -0 0, axis 0 0 1, limit lower=-0.84903 upper=0.87973 effort=10 velocity=3.14, mimic joint=lhand_joint multiplier=1.35269 offset=0
- joint lhand_joint: axis 0 0 1 -> 0 0 -1; child lhand_command_link -> lhand_small_needle_holder_link1_1; limit effort=2.0 velocity=6.8 -> lower=-0.62832 upper=0.62832 effort=10 velocity=3.14; origin xyz=0 0 0 rpy=0 0 0 -> xyz=7.9738e-05 0.006746875 0.013703058 rpy=-3.141592607 0 1.5707963; parent lhand_base_link -> lhand_xl_xc_330_1; type continuous -> revolute

File: jsk_hand/dynamixel_detachable_hand/urdf/rhand_detacher.urdf (robot description, URDF)
Before this commit: robot rhand_detacher_robot, 2 links, 1 joints
Links:
- removed link base_link
- added link rhand_base_link; visual box size=0.2 0.2 0.2
Joints:
- joint rhand_detach_joint_0: parent base_link -> rhand_base_link

File: jsk_hand/dynamixel_detachable_hand/urdf/rhand_gripper.urdf (robot description, URDF)
Before this commit: robot rhand_gripper_robot, 3 links, 2 joints
Links:
- removed link rhand_link
- added link rhand_bottom_spacer3300a_1, mass 0.00617072; collision mesh filename=package://dynamixel_detachable_hand/meshes/nejineji_finger_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; visual mesh filename=package://dynamixel_detachable_hand/meshes/nejineji_finger_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
- added link rhand_finger_11, mass 0.0442481; collision mesh filename=package://dynamixel_detachable_hand/meshes/nejineji_finger_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; visual mesh filename=package://dynamixel_detachable_hand/meshes/nejineji_finger_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
- added link rhand_finger_13, mass 0.0442481; collision mesh filename=package://dynamixel_detachable_hand/meshes/nejineji_finger_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; visual mesh filename=package://dynamixel_detachable_hand/meshes/nejineji_finger_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
- added link rhand_pinion_1, mass 0.00261444; collision mesh filename=package://dynamixel_detachable_hand/meshes/nejineji_finger_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; visual mesh filename=package://dynamixel_detachable_hand/meshes/nejineji_finger_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
- added link rhand_screwlock_male_1, mass 0.0103795; collision mesh filename=package://dynamixel_detachable_hand/meshes/nejineji_finger_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; visual mesh filename=package://dynamixel_detachable_hand/meshes/nejineji_finger_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
- added link rhand_small_diameter_hornb_1, mass 0.000682303; collision mesh filename=package://dynamixel_detachable_hand/meshes/nejineji_finger_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; visual mesh filename=package://dynamixel_detachable_hand/meshes/nejineji_finger_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
- added link rhand_tip_link
- added link rhand_xl_xc_330_1_2, mass 0.0168537; collision mesh filename=package://dynamixel_detachable_hand/meshes/nejineji_finger_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; visual mesh filename=package://dynamixel_detachable_hand/meshes/nejineji_finger_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
- link rhand_base_link: mass None -> 0.0498606; geometry collision mesh filename=package://dynamixel_detachable_hand/meshes/nejineji_finger_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; visual mesh filename=package://dynamixel_detachable_hand/meshes/nejineji_finger_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
Joints:
- added joint rhand_buttom_spacer3300a_1__screwlock_male_1: type fixed, parent rhand_bottom_spacer3300a_1, child rhand_screwlock_male_1, origin xyz=-5.6e-06 0.007707033 -0.003298772 rpy=0 -1.570796301 0, axis -0 1 -0
- added joint rhand_finger_mimic_joint: type prismatic, parent rhand_base_link, child rhand_finger_13, origin xyz=0 0 0 rpy=0 -0 0, axis -1 0 0, limit lower=-0.05 upper=0 effort=10 velocity=3.14, mimic joint=rhand_joint multiplier=-1 offset=0
- added joint rhand_servo_and_case_simple_1__pinion_1: type fixed, parent rhand_base_link, child rhand_pinion_1, origin xyz=-6.95e-06 -7.0943e-05 0.005234895 rpy=-3.141592607 0 -0.09765488, axis -0 0 -1
- added joint rhand_servo_and_case_simple_1__small_diameter_hornb_1: type fixed, parent rhand_base_link, child rhand_small_diameter_hornb_1, origin xyz=-5.065e-06 0 0.000967784 rpy=0 0 -3.141592607, axis 0 1 0
- added joint rhand_servo_and_case_simple_1__xl_xc_330_1_2: type fixed, parent rhand_base_link, child rhand_xl_xc_330_1_2, origin xyz=-0.0067468 7.9755e-05 -0.015702072 rpy=0 0 -1.5707963, axis 0 0 -1
- added joint rhand_to_tip: type fixed, parent rhand_base_link, child rhand_tip_link, origin xyz=0 0 0.06743 rpy=0 0 0
- added joint rhand_xl_xc_330_1_2__buttom_spacer3300a_1: type fixed, parent rhand_xl_xc_330_1_2, child rhand_bottom_spacer3300a_1, origin xyz=7.9799e-05 0.003444766 -0.015364374 rpy=-1.5707963 0 3.141592607, axis 0 -1 0
- joint rhand_joint: axis 0 1 0 -> -1 0 0; child rhand_link -> rhand_finger_11; limit effort=2.0 velocity=6.8 -> lower=0 upper=0.05 effort=2.0 velocity=0.1; origin xyz=0 0 0.1 rpy=0 0 0 -> xyz=0 0 0 rpy=0 -0 0; type continuous -> prismatic

File: jsk_hand/surgenoid_needle_holder_description/urdf/surgenoid_needle_holder_description.urdf (robot description, URDF)
Before this commit: robot rhand_needle_holder_robot, 8 links, 7 joints
Links:
- removed link rhand_base_link
- removed link rhand_detach_link_0
- removed link rhand_small_needle_holder_base_1
- removed link rhand_small_needle_holder_link1_1
- removed link rhand_small_needle_holder_link2_1
- removed link rhand_surgery_clamp_01_1
- removed link rhand_surgery_clamp_assy_1
- removed link rhand_xl_xc_330_1
- added link SURGERY_CLAMP_01_1, mass 0.00562524; collision mesh filename=package://surgenoid_needle_holder_description/meshes/SURGER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; visual mesh filename=package://surgenoid_needle_holder_description/meshes/SURGER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
- added link SURGERY_CLAMP_ASSY_1, mass 0.00675555; collision mesh filename=package://surgenoid_needle_holder_description/meshes/SURGER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; visual mesh filename=package://surgenoid_needle_holder_description/meshes/SURGER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
- added link XL_XC_330_1, mass 0.0168532; collision mesh filename=package://surgenoid_needle_holder_description/meshes/XL_XC_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; visual mesh filename=package://surgenoid_needle_holder_description/meshes/XL_XC_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
- added link base_link, mass 0.0162824; collision mesh filename=package://surgenoid_needle_holder_description/meshes/screwl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; visual mesh filename=package://surgenoid_needle_holder_description/meshes/screwl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
- added link small_needle_hoder_base_1, mass 0.020773; collision mesh filename=package://surgenoid_needle_holder_description/meshes/small_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; visual mesh filename=package://surgenoid_needle_holder_description/meshes/small_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
- added link small_needle_holder_link1_1, mass 0.00332751; collision mesh filename=package://surgenoid_needle_holder_description/meshes/small_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; visual mesh filename=package://surgenoid_needle_holder_description/meshes/small_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
- added link small_needle_holder_link2_1, mass 0.00195003; collision mesh filename=package://surgenoid_needle_holder_description/meshes/small_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; visual mesh filename=package://surgenoid_needle_holder_description/meshes/small_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
Joints:
- removed joint rhand_detach_joint_0
- removed joint rhand_holder_base_to_clamp
- removed joint rhand_holder_base_to_motor
- removed joint rhand_holder_jaw_joint
- removed joint rhand_holder_screw_to_base
- removed joint rhand_holder_tip_joint
- removed joint rhand_joint
- added joint SURGERY_CLAMP_ASSY_1__SURGERY_CLAMP_01_1: type revolute, parent SURGERY_CLAMP_ASSY_1, child SURGERY_CLAMP_01_1, origin xyz=0.040124645 -0.00714826 0.001320943 rpy=0 0 3.0922928, axis 0 0 -1, limit lower=-0.29662 upper=0.44772 effort=10 velocity=3.14, mimic joint=XL_XC_330_1__small_needle_holder_link1_1 multiplier=0.581031 offset=0
- added joint XL_XC_330_1__small_needle_holder_link1_1: type revolute, parent XL_XC_330_1, child small_needle_holder_link1_1, origin xyz=7.9738e-05 0.006746875 0.013703058 rpy=-3.141592607 0 1.5707963, axis 0 0 -1, limit lower=-0.62832 upper=0.62832 effort=10 velocity=3.14
- added joint screwlock_male_hard_v2_1__small_needle_hoder_base_1: type fixed, parent base_link, child small_needle_hoder_base_1, origin xyz=-0.009065668 -0.000168333 -0.015571405 rpy=-6.327e-06 -2.654e-06 3.141589, axis 0 0 1
- added joint small_needle_hoder_base_1__SURGERY_CLAMP_ASSY_1: type fixed, parent small_needle_hoder_base_1, child SURGERY_CLAMP_ASSY_1, origin xyz=-0.037277901 0.011289345 -0.004030915 rpy=0 0 -3.0922928, axis 0 0 -1
- added joint small_needle_hoder_base_1__XL_XC_330_1: type fixed, parent small_needle_hoder_base_1, child XL_XC_330_1, origin xyz=0.038688034 -0.006248738 0.011774486 rpy=-3.141592607 0 1.5707963, axis 0 0 -1
- added joint small_needle_holder_link1_1__small_needle_holder_link2_1: type revolute, parent small_needle_holder_link1_1, child small_needle_holder_link2_1, origin xyz=0.020772397 0.033007689 -0.017 rpy=0 -0 0, axis 0 0 1, limit lower=-0.84903 upper=0.87973 effort=10 velocity=3.14, mimic joint=XL_XC_330_1__small_needle_holder_link1_1 multiplier=1.35269 offset=0
